File: line-follower-robot-01.kicad_sch (KiCad schematic)
At the start: 47 parts, among them J1 Conn_01x02, J2 Conn_01x11, J3 Conn_01x02, J4 Conn_01x06, J5 Conn_01x02, J6 Conn_01x04, J7 Conn_01x05, SW1 SW_SPDT, SW2 SW_Push, U1 STM32F446RETx, U2 TB6612FNG, U3 LM1117DT-3.3, U4 TB6612FNG, U5 LM1117DT-5.0, Y1 8MHz

Commit message: changed some values, added disc boxes, added parts and part #
Parts:
- C1, C14, C16, C18, C22, C7: LCSC Part # (none) -> C19702
- C10, C11: value 16p -> 18p; LCSC Part # (none) -> C1647
- C15, C2, C3, C4, C5, C6, C8: LCSC Part # (none) -> C14663
- C9: LCSC Part # (none) -> C19666
- L1: value 27n -> 1u
- U1: LCSC Part # (none) -> C69336
- Y1: LCSC Part # (none) -> C57131
Other:
- moved on the sheet: J2, J4, J6, J7

Commit message: moved to pcb routing
Parts:
- removed L1: 1u, Inductor_SMD:L_0603_1608Metric_Pad1.05x0.95mm_HandSolder, symbol Device:L
- added C23: 1u, Capacitor_SMD:C_0603_1608Metric_Pad1.08x0.95mm_HandSolder, symbol Device:C
- added FB1: 120R, Inductor_SMD:L_0603_1608Metric_Pad1.05x0.95mm_HandSolder, symbol Device:FerriteBead
- added H1, H2, H3, H4: MountingHole, MountingHole:MountingHole_2.2mm_M2, symbol Mechanical:MountingHole
- added SW3: SW_Push, Button_Switch_SMD:SW_Push_1P1T_NO_CK_KSC7xxJ, symbol Switch:SW_Push
- C12, C13, C20, C21: LCSC Part # (none) -> C14663
- C17, C19: value 33u -> 10u; LCSC Part # (none) -> C19702
- C7: value 10u -> 1u
- D1: LCSC Part # (none) -> C2287
- D2, D4: LCSC Part # (none) -> C12624
- D3: LCSC Part # (none) -> C2286
- J2: footprint Connector_PinHeader_2.54mm:PinHeader_1x11_P2.54mm_Vertical -> Connector_PinHeader_2.54mm:PinHeader_1x11_P2.54mm_Horizontal; LCSC Part # (none) -> C725903
- R1: LCSC Part # (none) -> C177337
- R2, R3, R4, R5: LCSC Part # (none) -> C177343
- SW1: footprint Button_Switch_SMD:SW_SPDT_PCM12 -> Button_Switch_SMD:SW_SPDT_CK_JS102011SAQN; LCSC Part # (none) -> C221660
- SW2: footprint Button_Switch_SMD:SW_Push_1P1T_NO_E-Switch_TL3301NxxxxxG -> Button_Switch_SMD:SW_Push_1P1T_NO_CK_KSC7xxJ; LCSC Part # (none) -> C2799444
- U2, U4: LCSC Part # (none) -> C141517
- U3: value LM1117DT-3.3 -> LM1117MP-3.3; footprint Package_TO_SOT_SMD:TO-252-3_TabPin2 -> Package_TO_SOT_SMD:SOT-223-3_TabPin2; LCSC Part # (none) -> C3750685
- U5: value LM1117DT-5.0 -> LM1117MP-5.0; footprint Package_TO_SOT_SMD:TO-252-3_TabPin2 -> Package_TO_SOT_SMD:SOT-223-3_TabPin2; LCSC Part # (none) -> C498151
Connections:
- net +3.3V: now also C23.1, FB1.2; no longer J2.10 (Pin_10)
- net +3.3VA: now also FB1.1
- net +5V: now also J2.10 (Pin_10), J2.9 (Pin_9)
- net GND: now also C23.2, SW3.1
- net at U1.2 (PC13): now also SW3.2
- no-connect marks 26 -> 24
Other:
- note added: "+3.3V Regulation"
- note added: "+5V Regulation"
- note added: "1 x bulk decoupling + 100nF per VDD"
- note added: "Battery Connection"
- note added: "Computer UART"
- note added: "HC-05 Bluetooth UART"
- note added: "Mounting Holes"
- note added: "Programming SWD"
- note added: "QTR-8A Sensor"
- note added: "STM32F4 Microcontroller"
- note added: "TB6612FNG Motor Driver A"
- note added: "TB6612FNG Motor Driver B"
- note added: "low-pass filter for analog VDD"
- title: (none) -> line follower robot
- moved on the sheet: C7, C8, C9
