File: line-follower-robot-01.kicad_pcb (KiCad board)
At the start: 2 copper layers, 53 parts, among them J1 Conn_01x02, J2 Conn_01x11, J3 Conn_01x02, J4 Conn_01x06, J5 Conn_01x02, J6 Conn_01x04, J7 Conn_01x05, SW1 SW_SPDT, SW2 SW_Push, SW3 SW_Push, U1 STM32F446RETx, U2 TB6612FNG, U3 LM1117MP-3.3, U4 TB6612FNG, U5 LM1117MP-5.0, Y1 8MHz

Commit message: routing almost done
Parts:
- moved D1 36.3 mm to (113.4, 96.0)
- moved D2 34.5 mm to (109.8, 96.0)
- moved R2 32.3 mm to (113.4, 97.8)
- moved R3 30.5 mm to (110.0, 97.8)
- moved D3 12.7 mm to (93.1, 114.4), turned to 180 degrees
- moved R4 9.86 mm to (93.2, 112.5)
- moved D4 7.64 mm to (114.6, 117.3), turned to 180 degrees
- moved J6 4.97 mm to (97.1, 116.6)
- moved R5 3.85 mm to (110.8, 117.3), turned to 180 degrees
- moved C8 1.00 mm to (101.6, 107.4)
- moved C12 0.90 mm to (120.1, 125.3)
- moved C1 0.50 mm to (100.2, 100.7)
- moved C10 0.50 mm to (99.5, 104.3)
- moved C11 0.50 mm to (99.5, 107.8)
- moved C15 0.50 mm to (97.3, 101.6)
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Routing:
- net +3.3V: track 45.0 -> 245.1 mm, vias 0 -> 2
- net PB4: track 0.00 -> 48.8 mm, vias 0 -> 2
- net PB5: track 0.00 -> 40.3 mm, vias 0 -> 2
- net PC9: track 0.00 -> 37.9 mm, vias 0 -> 2
- net PC8: track 0.00 -> 35.2 mm, vias 0 -> 2
- net /RUN_BTN: track 0.00 -> 32.7 mm, vias 0 -> 2
- net PC1: track 0.00 -> 31.5 mm, vias 0 -> 1
- net PC6: track 0.00 -> 31.1 mm, vias 0 -> 2
- net Net-(U1-PC13): track 0.00 -> 28.6 mm, vias 0 -> 2
- net GND: track 62.1 -> 90.4 mm, vias 25 -> 40
- net Net-(U1-PC12): track 0.00 -> 26.9 mm, vias 0 -> 2
- net PC5: track 0.00 -> 26.8 mm, vias 0 -> 2
- net PB0: track 0.00 -> 24.2 mm, vias 0 -> 1
- net RESET: track 0.00 -> 24.2 mm, vias 0 -> 1
- net +5V: track 34.3 -> 57.9 mm
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